File: board/schemat.sch (EAGLE design)
At the start: 42 parts, among them IC1 MEGA8-P, IC2 L293D, Q1 10MHz

Commit message: Adding on github
Connections:
- removed net VCC_MOTOR: IC2.VCC2
- net VCC_MOTORS: now also IC2.VCC2
Changed lines of the file:
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@@
-</segment>
-</net>
-<net name="VCC_MOTOR" class="0">
-<segment>
-<pinref part="IC2" gate="G$1" pin="VCC2"/>
-<wire x1="-20.32" y1="-88.9" x2="-10.16" y2="-88.9" width="0.1524" layer="91"/>
-<label x="-20.32" y="-88.9" size="1.778" layer="95" rot="R180" xref="yes"/>
 </segment>
 </net>
@@
 <junction x="-15.24" y="0"/>
 </segment>
+<segment>
+<pinref part="IC2" gate="G$1" pin="VCC2"/>
+<wire x1="-20.32" y1="-88.9" x2="-10.16" y2="-88.9" width="0.1524" layer="91"/>
+<label x="-20.32" y="-88.9" size="1.778" layer="95" rot="R180" xref="yes"/>
+</segment>
 </net>
